Commit message: Add state publisher

File: urdf/turtlebro.urdf (robot description, URDF)
Before this commit: robot turtlebro, 1 links, 0 joints
Links:
- added link base_footprint
- added link base_scan, mass 0.114; collision cylinder length=0.0315 radius=0.055; visual cylinder length=0.0315 radius=0.055
Joints:
- added joint base_joint: type fixed, parent base_footprint, child base_link, origin xyz=0.0 0.0 0.010 rpy=0 0 0
- added joint scan_joint: type fixed, parent base_link, child base_scan, origin xyz=0.0 0 0.05 rpy=0 0 0

Commit message: fix laser frame

File: urdf/turtlebro.urdf (robot description, URDF)
Before this commit: robot turtlebro, 3 links, 2 joints
Joints:
- joint scan_joint: origin xyz=0.0 0 0.05 rpy=0 0 0 -> xyz=0.0 0 0.05 rpy=0 0 3.1415

Commit message: play with URDF

File: urdf/turtlebro.urdf (robot description, URDF)
Before this commit: robot turtlebro, 3 links, 2 joints
Links:
- added link imu_link; visual box size=0.18 0.18 0.002
Joints:
- added joint imu_joint: type fixed, parent base_link, child imu_link, origin xyz=0.0 0 0.025 rpy=0 0 0
- joint base_joint: origin xyz=0.0 0.0 0.010 rpy=0 0 0 -> xyz=0.0 0.0 0.025 rpy=0 0 0
- joint scan_joint: origin xyz=0.0 0 0.05 rpy=0 0 3.1415 -> xyz=0.0 0 0.08 rpy=0 0 3.1415

Commit message: Whels at model

File: urdf/turtlebro.urdf (robot description, URDF)
Before this commit: robot turtlebro, 4 links, 3 joints
Links:
- added link wheel_left_link; visual cylinder length=0.025 radius=0.03
- added link wheel_right_link; visual cylinder length=0.025 radius=0.03
- link base_scan: mass 0.114 -> None; geometry visual cylinder length=0.0515 radius=0.055
Joints:
- added joint wheel_left_joint: type fixed, parent base_link, child wheel_left_link, origin xyz=0 0.115 0 rpy=0 0 0, axis 0 0 1
- added joint wheel_right_joint: type fixed, parent base_link, child wheel_right_link, origin xyz=0 -0.115 0 rpy=0 0 0, axis 0 0 1
- joint imu_joint: origin xyz=0.0 0 0.025 rpy=0 0 0 -> xyz=0.0 0 0.035 rpy=0 0 0

Commit message: Update turtlebro.urdf
scan link adjusted

File: urdf/turtlebro.urdf (robot description, URDF)
Before this commit: robot turtlebro, 6 links, 5 joints
Links:
- link base_scan: geometry visual cylinder length=0.0515 radius=0.035
